Commit message: Update ball_beam.urdf

File: ball_beam.urdf (robot description, URDF)
Before this commit: robot simplecar, 7 links, 6 joints
Joints:
- joint left_track_center_beam: type static -> fixed
- joint right_track_center_beam: type static -> fixed
- joint stopper_to_center_beam: type static -> fixed
