Commit message: moves continuously in the opposite direction

File: simple_beam.urdf (robot description, URDF)
Before this commit: robot simplebeam, 4 links, 3 joints
Links:
- link center_beam: mass 0.5 -> 1
Joints:
- joint rod_to_left_hinge: limit lower=-0.5 upper=0.5 effort=100 velocity=100 -> (none); type revolute -> continuous

Commit message: working sim

File: simple_beam.urdf (robot description, URDF)
Before this commit: robot simplebeam, 4 links, 3 joints
Links:
- removed link left_hinge
Joints:
- removed joint hinge_to_center_beam
- removed joint rod_to_left_hinge
- added joint rod_to_center_beam: type continuous, parent left_rod, child center_beam, origin xyz=0 0 .1, axis 0 1 0, limit lower=-0.5 upper=0.5 effort=100 velocity=100

Commit message: working sim

File: simple_beam.urdf (robot description, URDF)
Before this commit: robot simplebeam, 3 links, 2 joints
Joints:
- joint rod_to_center_beam: limit lower=-0.5 upper=0.5 effort=100 velocity=100 -> lower=-0.5 upper=0.25 effort=100 velocity=100
